File: docs/nrf_glider/glider_rx.sch (KiCad schematic (older format))
At the start: 8 parts, among them J5 Conn_01x12_Female, M1 Servo Left, M2 Servo Right, U5 LM1117-3.3

Commit message: Rerouted Rx module for center buzzer
Parts:
- removed J5: Conn_01x12_Female, Connector_PinHeader_2.54mm:PinHeader_1x12_P2.54mm_Vertical, symbol Connector:Conn_01x12_Female
- added J7, J8: Conn_01x06_Female, Connector_PinHeader_2.54mm:PinHeader_1x06_P2.54mm_Vertical, symbol Connector:Conn_01x06_Female
- U5: footprint (none) -> Package_TO_SOT_THT:TO-220-3_Horizontal_TabDown
Connections:
- wire segments 23 -> 25
Other:
- moved on the sheet: BT2, BZ2
Changed lines of the file:
@@
 EESchema Schematic File Version 4
-LIBS:nrf_glider-cache
+LIBS:glider_rx-cache
 EELAYER 26 0
 EELAYER END
 $Descr A4 11693 8268
 encoding utf-8
-Sheet 1 5
+Sheet 1 1
 Title ""
 Date ""
@@
 F 0 "U5" H 4500 2092 50  0000 C CNN
 F 1 "LM1117-3.3" H 4500 2001 50  0000 C CNN
-F 2 "" H 4500 1850 50  0001 C CNN
+F 2 "Package_TO_SOT_THT:TO-220-3_Horizontal_TabDown" H 4500 1850 50  0001 C CNN
 F 3 "http://www.ti.com/lit/ds/symlink/lm1117.pdf" H 4500 1850 50  0001 C CNN
 	1    4500 1850
@@
 $EndComp
 $Comp
-L power:GND #PWR0129
+L power:GND #PWR035
 U 1 1 5BCED801
-P 4500 2150
-F 0 "#PWR0129" H 4500 1900 50  0001 C CNN
-F 1 "GND" H 4505 1977 50  0000 C CNN
-F 2 "" H 4500 2150 50  0001 C CNN
-F 3 "" H 4500 2150 50  0001 C CNN
-	1    4500 2150
+P 4500 2300
+F 0 "#PWR035" H 4500 2050 50  0001 C CNN
+F 1 "GND" H 4505 2127 50  0000 C CNN
+F 2 "" H 4500 2300 50  0001 C CNN
+F 3 "" H 4500 2300 50  0001 C CNN
+	1    4500 2300
 	1    0    0    -1
 $EndComp
@@
 L Device:Battery BT2
 U 1 1 5BCED8B9
-P 3700 2050
-F 0 "BT2" H 3808 2096 50  0000 L CNN
-F 1 "4.5V - 9.9V" H 3808 2005 50  0000 L CNN
-F 2 "Connector_PinHeader_2.54mm:PinHeader_1x02_P2.54mm_Vertical" V 3700 2110 50  0001 C CNN
-F 3 "~" V 3700 2110 50  0001 C CNN
-	1    3700 2050
-	1    0    0    -1
-$EndComp
-Wire Wire Line
-	3700 1850 4200 1850
-$Comp
-L power:GND #PWR0130
+P 3100 1950
+F 0 "BT2" H 3208 1996 50  0000 L CNN
+F 1 "4.5V - 9.9V" H 3208 1905 50  0000 L CNN
+F 2 "Connector_PinHeader_2.54mm:PinHeader_1x02_P2.54mm_Vertical" V 3100 2010 50  0001 C CNN
+F 3 "~" V 3100 2010 50  0001 C CNN
+	1    3100 1950
+	1    0    0    -1
+$EndComp
+$Comp
+L power:GND #PWR030
 U 1 1 5BCED983
-P 3700 2250
-F 0 "#PWR0130" H 3700 2000 50  0001 C CNN
-F 1 "GND" H 3705 2077 50  0000 C CNN
-F 2 "" H 3700 2250 50  0001 C CNN
-F 3 "" H 3700 2250 50  0001 C CNN
-	1    3700 2250
-	1    0    0    -1
-$EndComp
-$Comp
-L power:VCC #PWR0131
+P 3100 2150
+F 0 "#PWR030" H 3100 1900 50  0001 C CNN
+F 1 "GND" H 3105 1977 50  0000 C CNN
+F 2 "" H 3100 2150 50  0001 C CNN
+F 3 "" H 3100 2150 50  0001 C CNN
+	1    3100 2150
+	1    0    0    -1
+$EndComp
+$Comp
+L power:VCC #PWR039
 U 1 1 5BCED9FA
 P 5350 1850
-F 0 "#PWR0131" H 5350 1700 50  0001 C CNN
+F 0 "#PWR039" H 5350 1700 50  0001 C CNN
 F 1 "VCC" H 5367 2023 50  0000 C CNN
 F 2 "" H 5350 1850 50  0001 C CNN
@@
 $EndComp
 $Comp
-L power:GND #PWR0132
+L power:GND #PWR038
 U 1 1 5BCEDF2F
 P 4900 2150
-F 0 "#PWR0132" H 4900 1900 50  0001 C CNN
+F 0 "#PWR038" H 4900 1900 50  0001 C CNN
 F 1 "GND" H 4905 1977 50  0000 C CNN
 F 2 "" H 4900 2150 50  0001 C CNN
@@
 $EndComp
 $Comp
-L power:GND #PWR0133
+L power:GND #PWR040
 U 1 1 5BCEDF6D
 P 5350 2100
-F 0 "#PWR0133" H 5350 1850 50  0001 C CNN
+F 0 "#PWR040" H 5350 1850 50  0001 C CNN
 F 1 "GND" H 5355 1927 50  0000 C CNN
 F 2 "" H 5350 2100 50  0001 C CNN
@@
 	4800 1850 4900 1850
 $Comp
-L power:VDD #PWR0134
+L power:VDD #PWR029
 U 1 1 5BCF6415
-P 3700 1850
-F 0 "#PWR0134" H 3700 1700 50  0001 C CNN
-F 1 "VDD" H 3717 2023 50  0000 C CNN
-F 2 "" H 3700 1850 50  0001 C CNN
-F 3 "" H 3700 1850 50  0001 C CNN
-	1    3700 1850
-	1    0    0    -1
-$EndComp
-Connection ~ 3700 1850
+P 3100 1750
+F 0 "#PWR029" H 3100 1600 50  0001 C CNN
+F 1 "VDD" H 3117 1923 50  0000 C CNN
+F 2 "" H 3100 1750 50  0001 C CNN
+F 3 "" H 3100 1750 50  0001 C CNN
+	1    3100 1750
+	1    0    0    -1
+$EndComp
 Wire Wire Line
 	5350 1850 5350 1900
@@
 Connection ~ 4900 1850
 $Comp
-L Connector:Conn_01x12_Female J5
-U 1 1 5BD137AB
-P 3250 3750
-F 0 "J5" H 3144 4435 50  0000 C CNN
-F 1 "Conn_01x12_Female" H 3144 4344 50  0000 C CNN
-F 2 "Connector_PinHeader_2.54mm:PinHeader_1x12_P2.54mm_Vertical" H 3250 3750 50  0001 C CNN
-F 3 "~" H 3250 3750 50  0001 C CNN
-	1    3250 3750
-	-1   0    0    -1
-$EndComp
-$Comp
-L power:VDD #PWR0135
+L power:VDD #PWR032
 U 1 1 5BD1962D
 P 3900 3250
-F 0 "#PWR0135" H 3900 3100 50  0001 C CNN
+F 0 "#PWR032" H 3900 3100 50  0001 C CNN
 F 1 "VDD" H 3917 3423 50  0000 C CNN
 F 2 "" H 3900 3250 50  0001 C CNN
@@
 	3900 3250 3450 3250
 $Comp
-L power:VCC #PWR0136
+L power:VCC #PWR034
 U 1 1 5BD1B4CC
 P 4100 3350
-F 0 "#PWR0136" H 4100 3200 50  0001 C CNN
+F 0 "#PWR034" H 4100 3200 50  0001 C CNN
 F 1 "VCC" H 4117 3523 50  0000 C CNN
 F 2 "" H 4100 3350 50  0001 C CNN
@@
 	3450 3350 4100 3350
 $Comp
-L power:GND #PWR0137
+L power:GND #PWR031
 U 1 1 5BD1F411
-P 3550 4350
-F 0 "#PWR0137" H 3550 4100 50  0001 C CNN
-F 1 "GND" H 3555 4177 50  0000 C CNN
-F 2 "" H 3550 4350 50  0001 C CNN
-F 3 "" H 3550 4350 50  0001 C CNN
-	1    3550 4350
-	1    0    0    -1
-$EndComp
-Wire Wire Line
-	3450 4350 3550 4350
+P 3600 4550
+F 0 "#PWR031" H 3600 4300 50  0001 C CNN
+F 1 "GND" H 3605 4377 50  0000 C CNN
+F 2 "" H 3600 4550 50  0001 C CNN
+F 3 "" H 3600 4550 50  0001 C CNN
+	1    3600 4550
+	1    0    0    -1
+$EndComp
+Wire Wire Line
+	3500 4550 3600 4550
 $Comp
 L Motor:Motor_Servo M1
@@
 L Device:Buzzer BZ2
 U 1 1 5BD29AB3
-P 4100 4350
-F 0 "BZ2" H 4253 4379 50  0000 L CNN
-F 1 "Buzzer" H 4253 4288 50  0000 L CNN
-F 2 "Buzzer_Beeper:Buzzer_15x7.5RM7.6" V 4075 4450 50  0001 C CNN
-F 3 "~" V 4075 4450 50  0001 C CNN
-	1    4100 4350
+P 4150 4550
+F 0 "BZ2" H 4303 4579 50  0000 L CNN
+F 1 "Buzzer" H 4303 4488 50  0000 L CNN
+F 2 "Buzzer_Beeper:Buzzer_15x7.5RM7.6" V 4125 4650 50  0001 C CNN
+F 3 "~" V 4125 4650 50  0001 C CNN
+	1    4150 4550
 	1    0    0    -1
 $EndComp
@@
 	4450 4000 4900 4000
 $Comp
-L power:VDD #PWR0138
+L power:VDD #PWR037
 U 1 1 5BD6892B
 P 4750 3400
-F 0 "#PWR0138" H 4750 3250 50  0001 C CNN
+F 0 "#PWR037" H 4750 3250 50  0001 C CNN
 F 1 "VDD" H 4767 3573 50  0000 C CNN
 F 2 "" H 4750 3400 50  0001 C CNN
@@
 Connection ~ 4750 3600
 $Comp
-L power:GND #PWR0139
+L power:GND #PWR036
 U 1 1 5BD6F7A2
 P 4600 4400
-F 0 "#PWR0139" H 4600 4150 50  0001 C CNN
+F 0 "#PWR036" H 4600 4150 50  0001 C CNN
 F 1 "GND" H 4605 4227 50  0000 C CNN
 F 2 "" H 4600 4400 50  0001 C CNN
@@
 	4600 3700 4900 3700
 Connection ~ 4600 4200
-Wire Wire Line
-	3450 4250 4000 4250
-$Comp
-L power:GND #PWR0140
+$Comp
+L power:GND #PWR033
 U 1 1 5BD8512D
-P 4000 4500
-F 0 "#PWR0140" H 4000 4250 50  0001 C CNN
-F 1 "GND" H 4005 4327 50  0000 C CNN
-F 2 "" H 4000 4500 50  0001 C CNN
-F 3 "" H 4000 4500 50  0001 C CNN
-	1    4000 4500
-	1    0    0    -1
-$EndComp
-Wire Wire Line
-	4000 4450 4000 4500
+P 4050 4700
+F 0 "#PWR033" H 4050 4450 50  0001 C CNN
+F 1 "GND" H 4055 4527 50  0000 C CNN
+F 2 "" H 4050 4700 50  0001 C CNN
+F 3 "" H 4050 4700 50  0001 C CNN
+	1    4050 4700
+	1    0    0    -1
+$EndComp
+Wire Wire Line
+	4050 4650 4050 4700
 Text Notes 7400 7500 0    50   ~ 0
 NRF and MSP430 based RC control
@@
 Text HLabel 3250 3750 0    50   BiDi ~ 0
 A3
-Text HLabel 3250 3850 0    50   BiDi ~ 0
+Text HLabel 3300 4050 0    50   BiDi ~ 0
 IO0
-Text HLabel 3250 3950 0    50   BiDi ~ 0
+Text HLabel 3300 4150 0    50   BiDi ~ 0
 IO1
-Text HLabel 3250 4050 0    50   BiDi ~ 0
+Text HLabel 3300 4250 0    50   BiDi ~ 0
 IO2
-Text HLabel 3250 4150 0    50   BiDi ~ 0
+Text HLabel 3300 4350 0    50   BiDi ~ 0
 IO3
-Text HLabel 3250 4250 0    50   BiDi ~ 0
+Text HLabel 3300 4450 0    50   BiDi ~ 0
 IO4
-Text HLabel 3250 4350 0    50   Output ~ 0
+Text HLabel 3300 4550 0    50   Output ~ 0
 GND
+$Comp
+L Connector:Conn_01x06_Female J7
+U 1 1 5BE9CBB2
+P 3250 3450
+F 0 "J7" H 3144 3835 50  0000 C CNN
+F 1 "Conn_01x06_Female" H 3144 3744 50  0000 C CNN
+F 2 "Connector_PinHeader_2.54mm:PinHeader_1x06_P2.54mm_Vertical" H 3250 3450 50  0001 C CNN
+F 3 "~" H 3250 3450 50  0001 C CNN
+	1    3250 3450
+	-1   0    0    -1
+$EndComp
+$Comp
+L Connector:Conn_01x06_Female J8
+U 1 1 5BE9DA2D
+P 3300 4250
+F 0 "J8" H 3194 4635 50  0000 C CNN
+F 1 "Conn_01x06_Female" H 3194 4544 50  0000 C CNN
+F 2 "Connector_PinHeader_2.54mm:PinHeader_1x06_P2.54mm_Vertical" H 3300 4250 50  0001 C CNN
+F 3 "~" H 3300 4250 50  0001 C CNN
+	1    3300 4250
+	-1   0    0    -1
+$EndComp
+Wire Wire Line
+	4500 2150 4500 2300
+Wire Wire Line
+	4200 1850 4200 1750
+Wire Wire Line
+	4200 1750 3100 1750
+Connection ~ 3100 1750
+Wire Wire Line
+	3500 4450 4050 4450
 $EndSCHEMATC
