File: docs/nrf_glider/glider_tx.sch (KiCad schematic (older format))
At the start: 12 parts, among them J3 UART, J4 Conn_01x12_Female, SW1 SW_SPST, SW2 TRIM, U4 LM1117-3.3

Commit message: Rerouted Rx module for center buzzer
Parts:
- removed J4: Conn_01x12_Female, Connector_PinHeader_2.54mm:PinHeader_1x12_P2.54mm_Vertical, symbol Connector:Conn_01x12_Female
- added BZ2: Buzzer, symbol Device:Buzzer
- added J4, J6: Conn_01x06_Female, Connector_PinHeader_2.54mm:PinHeader_1x06_P2.54mm_Vertical, symbol Connector:Conn_01x06_Female
- SW1: footprint (none) -> Button_Switch_SMD:SW_SPST_SKQG_WithStem
- U4: footprint (none) -> Package_TO_SOT_THT:TO-220-3_Horizontal_TabDown
- renumbered J3 to J5
Connections:
- wire segments 40 -> 52
Changed lines of the file:
@@
 EESchema Schematic File Version 4
-LIBS:nrf_glider-cache
+LIBS:glider_tx-cache
 EELAYER 26 0
 EELAYER END
 $Descr A4 11693 8268
 encoding utf-8
-Sheet 3 5
+Sheet 1 1
 Title ""
 Date ""
@@
 $EndDescr
 $Comp
-L Connector:Conn_01x12_Female J4
-U 1 1 5BD138DF
-P 4150 3750
-F 0 "J4" H 4044 4435 50  0000 C CNN
-F 1 "Conn_01x12_Female" H 4044 4344 50  0000 C CNN
-F 2 "Connector_PinHeader_2.54mm:PinHeader_1x12_P2.54mm_Vertical" H 4150 3750 50  0001 C CNN
-F 3 "~" H 4150 3750 50  0001 C CNN
-	1    4150 3750
-	-1   0    0    -1
-$EndComp
-$Comp
-L power:VCC #PWR0114
+L power:VCC #PWR019
 U 1 1 5BD1D3CE
 P 5150 3150
-F 0 "#PWR0114" H 5150 3000 50  0001 C CNN
+F 0 "#PWR019" H 5150 3000 50  0001 C CNN
 F 1 "VCC" H 5167 3323 50  0000 C CNN
 F 2 "" H 5150 3150 50  0001 C CNN
@@
 $EndComp
 $Comp
-L power:VDD #PWR0115
+L power:VDD #PWR017
 U 1 1 5BD1D429
 P 5000 2900
-F 0 "#PWR0115" H 5000 2750 50  0001 C CNN
+F 0 "#PWR017" H 5000 2750 50  0001 C CNN
 F 1 "VDD" H 5017 3073 50  0000 C CNN
 F 2 "" H 5000 2900 50  0001 C CNN
@@
 $EndComp
 $Comp
-L power:GND #PWR0116
+L power:GND #PWR015
 U 1 1 5BD1F482
 P 4450 4350
-F 0 "#PWR0116" H 4450 4100 50  0001 C CNN
+F 0 "#PWR015" H 4450 4100 50  0001 C CNN
 F 1 "GND" H 4455 4177 50  0000 C CNN
 F 2 "" H 4450 4350 50  0001 C CNN
@@
 F 0 "U4" H 6300 1692 50  0000 C CNN
 F 1 "LM1117-3.3" H 6300 1601 50  0000 C CNN
-F 2 "" H 6300 1450 50  0001 C CNN
+F 2 "Package_TO_SOT_THT:TO-220-3_Horizontal_TabDown" H 6300 1450 50  0001 C CNN
 F 3 "http://www.ti.com/lit/ds/symlink/lm1117.pdf" H 6300 1450 50  0001 C CNN
 	1    6300 1450
@@
 $EndComp
 $Comp
-L power:GND #PWR0117
+L power:GND #PWR023
 U 1 1 5BD2C86D
 P 6300 1750
-F 0 "#PWR0117" H 6300 1500 50  0001 C CNN
+F 0 "#PWR023" H 6300 1500 50  0001 C CNN
 F 1 "GND" H 6305 1577 50  0000 C CNN
 F 2 "" H 6300 1750 50  0001 C CNN
@@
 $EndComp
 $Comp
-L power:GND #PWR0118
+L power:GND #PWR020
 U 1 1 5BD2C87B
 P 5500 1850
-F 0 "#PWR0118" H 5500 1600 50  0001 C CNN
+F 0 "#PWR020" H 5500 1600 50  0001 C CNN
 F 1 "GND" H 5505 1677 50  0000 C CNN
 F 2 "" H 5500 1850 50  0001 C CNN
@@
 $EndComp
 $Comp
-L power:VCC #PWR0119
+L power:VCC #PWR027
 U 1 1 5BD2C881
 P 7150 1450
-F 0 "#PWR0119" H 7150 1300 50  0001 C CNN
+F 0 "#PWR027" H 7150 1300 50  0001 C CNN
 F 1 "VCC" H 7167 1623 50  0000 C CNN
 F 2 "" H 7150 1450 50  0001 C CNN
@@
 $EndComp
 $Comp
-L power:GND #PWR0120
+L power:GND #PWR025
 U 1 1 5BD2C895
 P 6700 1750
-F 0 "#PWR0120" H 6700 1500 50  0001 C CNN
+F 0 "#PWR025" H 6700 1500 50  0001 C CNN
 F 1 "GND" H 6705 1577 50  0000 C CNN
 F 2 "" H 6700 1750 50  0001 C CNN
@@
 $EndComp
 $Comp
-L power:GND #PWR0121
+L power:GND #PWR028
 U 1 1 5BD2C89B
 P 7150 1700
-F 0 "#PWR0121" H 7150 1450 50  0001 C CNN
+F 0 "#PWR028" H 7150 1450 50  0001 C CNN
 F 1 "GND" H 7155 1527 50  0000 C CNN
 F 2 "" H 7150 1700 50  0001 C CNN
@@
 	6600 1450 6700 1450
 $Comp
-L power:VDD #PWR0122
+L power:VDD #PWR021
 U 1 1 5BD2C8A2
 P 6000 1350
-F 0 "#PWR0122" H 6000 1200 50  0001 C CNN
+F 0 "#PWR021" H 6000 1200 50  0001 C CNN
 F 1 "VDD" H 6017 1523 50  0000 C CNN
 F 2 "" H 6000 1350 50  0001 C CNN
@@
 	6700 1450 7150 1450
 Connection ~ 6700 1450
-Wire Wire Line
-	4350 4250 4900 4250
-$Comp
-L power:GND #PWR0123
+$Comp
+L power:GND #PWR016
 U 1 1 5BD90917
-P 4900 4550
-F 0 "#PWR0123" H 4900 4300 50  0001 C CNN
-F 1 "GND" H 4905 4377 50  0000 C CNN
-F 2 "" H 4900 4550 50  0001 C CNN
-F 3 "" H 4900 4550 50  0001 C CNN
-	1    4900 4550
-	1    0    0    -1
-$EndComp
-Wire Wire Line
-	4900 4450 4900 4550
+P 4900 4650
+F 0 "#PWR016" H 4900 4400 50  0001 C CNN
+F 1 "GND" H 4905 4477 50  0000 C CNN
+F 2 "" H 4900 4650 50  0001 C CNN
+F 3 "" H 4900 4650 50  0001 C CNN
+	1    4900 4650
+	1    0    0    -1
+$EndComp
 Wire Wire Line
 	4350 3450 5700 3450
@@
 	5800 4000 5900 4000
 $Comp
-L power:VCC #PWR0124
+L power:VCC #PWR026
 U 1 1 5BDA8B66
 P 6700 3250
-F 0 "#PWR0124" H 6700 3100 50  0001 C CNN
+F 0 "#PWR026" H 6700 3100 50  0001 C CNN
 F 1 "VCC" H 6717 3423 50  0000 C CNN
 F 2 "" H 6700 3250 50  0001 C CNN
@@
 Connection ~ 6700 3350
 $Comp
-L power:GND #PWR0125
+L power:GND #PWR024
 U 1 1 5BDB1721
 P 6650 4250
-F 0 "#PWR0125" H 6650 4000 50  0001 C CNN
+F 0 "#PWR024" H 6650 4000 50  0001 C CNN
 F 1 "GND" H 6655 4077 50  0000 C CNN
 F 2 "" H 6650 4250 50  0001 C CNN
@@
 Connection ~ 6650 4150
 $Comp
-L power:GND #PWR0126
+L power:GND #PWR022
 U 1 1 5BDC42C6
 P 6050 4600
-F 0 "#PWR0126" H 6050 4350 50  0001 C CNN
+F 0 "#PWR022" H 6050 4350 50  0001 C CNN
 F 1 "GND" H 6055 4427 50  0000 C CNN
 F 2 "" H 6050 4600 50  0001 C CNN
@@
 $EndComp
 $Comp
-L power:VCC #PWR0127
+L power:VCC #PWR018
 U 1 1 5BDCDC3B
 P 5100 3700
-F 0 "#PWR0127" H 5100 3550 50  0001 C CNN
+F 0 "#PWR018" H 5100 3550 50  0001 C CNN
 F 1 "VCC" H 5117 3873 50  0000 C CNN
 F 2 "" H 5100 3700 50  0001 C CNN
@@
 $EndComp
 $Comp
-L Connector:Conn_01x03_Male J3
+L Connector:Conn_01x03_Male J5
 U 1 1 5BCF8F2B
 P 4150 2500
-F 0 "J3" H 4256 2778 50  0000 C CNN
+F 0 "J5" H 4256 2778 50  0000 C CNN
 F 1 "UART" H 4256 2687 50  0000 C CNN
 F 2 "Connector_PinHeader_2.54mm:PinHeader_1x03_P2.54mm_Horizontal" H 4150 2500 50  0001 C CNN
@@
 	4700 3650 4350 3650
 $Comp
-L power:GND #PWR0128
+L power:GND #PWR014
 U 1 1 5BD038ED
 P 4450 2700
-F 0 "#PWR0128" H 4450 2450 50  0001 C CNN
+F 0 "#PWR014" H 4450 2450 50  0001 C CNN
 F 1 "GND" H 4455 2527 50  0000 C CNN
 F 2 "" H 4450 2700 50  0001 C CNN
@@
 Up/Down
 Wire Wire Line
-	4350 4150 5100 4150
-Wire Wire Line
 	5100 3700 5100 3800
 Wire Wire Line
@@
 F 0 "SW1" H 5700 1685 50  0000 C CNN
 F 1 "SW_SPST" H 5700 1594 50  0000 C CNN
-F 2 "" H 5700 1450 50  0001 C CNN
+F 2 "Button_Switch_SMD:SW_SPST_SKQG_WithStem" H 5700 1450 50  0001 C CNN
 F 3 "" H 5700 1450 50  0001 C CNN
 	1    5700 1450
@@
 Text HLabel 4150 3750 0    50   BiDi ~ 0
 A3
-Text HLabel 4150 3850 0    50   BiDi ~ 0
+Text HLabel 3900 4050 0    50   BiDi ~ 0
 IO0
-Text HLabel 4150 3950 0    50   BiDi ~ 0
+Text HLabel 3900 4150 0    50   BiDi ~ 0
 IO1
-Text HLabel 4150 4050 0    50   BiDi ~ 0
+Text HLabel 3900 4250 0    50   BiDi ~ 0
 IO2
-Text HLabel 4150 4150 0    50   BiDi ~ 0
+Text HLabel 3900 4350 0    50   BiDi ~ 0
 IO3
-Text HLabel 4150 4250 0    50   BiDi ~ 0
+Text HLabel 3900 4450 0    50   BiDi ~ 0
 IO4
-Text HLabel 4150 4350 0    50   Output ~ 0
+Text HLabel 3900 4550 0    50   Output ~ 0
 GND
+$Comp
+L Connector:Conn_01x06_Female J6
+U 1 1 5BE9EDB9
+P 4150 3450
+F 0 "J6" H 4044 3835 50  0000 C CNN
+F 1 "Conn_01x06_Female" H 4044 3744 50  0000 C CNN
+F 2 "Connector_PinHeader_2.54mm:PinHeader_1x06_P2.54mm_Vertical" H 4150 3450 50  0001 C CNN
+F 3 "~" H 4150 3450 50  0001 C CNN
+	1    4150 3450
+	-1   0    0    -1
+$EndComp
+$Comp
+L Connector:Conn_01x06_Female J4
+U 1 1 5BE9FD1D
+P 3900 4250
+F 0 "J4" H 3794 4635 50  0000 C CNN
+F 1 "Conn_01x06_Female" H 3794 4544 50  0000 C CNN
+F 2 "Connector_PinHeader_2.54mm:PinHeader_1x06_P2.54mm_Vertical" H 3900 4250 50  0001 C CNN
+F 3 "~" H 3900 4250 50  0001 C CNN
+	1    3900 4250
+	-1   0    0    -1
+$EndComp
+Wire Wire Line
+	4050 4550 4100 4550
+Connection ~ 4100 4550
+Wire Wire Line
+	4100 4550 4350 4550
+Wire Wire Line
+	4350 4550 4350 4350
+Wire Wire Line
+	4100 4450 4300 4450
+Wire Wire Line
+	4300 4450 4300 4250
+Wire Wire Line
+	4300 4250 4650 4250
+Wire Wire Line
+	4250 4150 4250 4350
+Wire Wire Line
+	4250 4350 4100 4350
+Wire Wire Line
+	4250 4150 5100 4150
+$Comp
+L Device:Buzzer BZ2
+U 1 1 5BEB1351
+P 4750 4450
+F 0 "BZ2" H 4903 4479 50  0000 L CNN
+F 1 "Buzzer" H 4903 4388 50  0000 L CNN
+F 2 "" V 4725 4550 50  0001 C CNN
+F 3 "~" V 4725 4550 50  0001 C CNN
+	1    4750 4450
+	1    0    0    -1
+$EndComp
+Wire Wire Line
+	4900 4450 4900 4600
+Wire Wire Line
+	4650 4550 4650 4600
+Wire Wire Line
+	4650 4600 4900 4600
+Connection ~ 4900 4600
+Wire Wire Line
+	4900 4600 4900 4650
+Wire Wire Line
+	4650 4350 4650 4250
+Connection ~ 4650 4250
+Wire Wire Line
+	4650 4250 4900 4250
 $EndSCHEMATC

Commit message: Added a TX2 which only has a header for the joystick and no switch on psu
Parts:
- removed BZ2: Buzzer, symbol Device:Buzzer
Connections:
- wire segments 52 -> 47
Changed lines of the file:
@@
 	4300 4450 4300 4250
-Wire Wire Line
-	4300 4250 4650 4250
 Wire Wire Line
 	4250 4150 4250 4350
@@
 Wire Wire Line
 	4250 4150 5100 4150
-$Comp
-L Device:Buzzer BZ2
-U 1 1 5BEB1351
-P 4750 4450
-F 0 "BZ2" H 4903 4479 50  0000 L CNN
-F 1 "Buzzer" H 4903 4388 50  0000 L CNN
-F 2 "" V 4725 4550 50  0001 C CNN
-F 3 "~" V 4725 4550 50  0001 C CNN
-	1    4750 4450
-	1    0    0    -1
-$EndComp
 Wire Wire Line
-	4900 4450 4900 4600
+	4900 4450 4900 4650
 Wire Wire Line
-	4650 4550 4650 4600
-Wire Wire Line
-	4650 4600 4900 4600
-Connection ~ 4900 4600
-Wire Wire Line
-	4900 4600 4900 4650
-Wire Wire Line
-	4650 4350 4650 4250
-Connection ~ 4650 4250
-Wire Wire Line
-	4650 4250 4900 4250
+	4300 4250 4900 4250
 $EndSCHEMATC
